File: KiCad/ESP32-S3-IO-DEVICE/ESP32-S3-IO-DEVICE.kicad_pcb (KiCad board)
At the start: 2 copper layers, 110 x 100 mm, 62 parts, among them J1 Terminal_04, J2 Terminal_04, J3 Terminal_06, J4 Terminal_02, J5 Terminal_04, J6 Terminal_06, Q1 2SC1815, Q10 2SC1815, Q11 2SC1815, Q12 2SC1815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

Commit message: Update schematic: fix wiring errors and improve component labeling
Parts:
- removed R1, R2: 10kΩ, Resistor_THT:R_Axial_DIN0207_L6.3mm_D2.5mm_P7.62mm_Horizontal
Connections:
- RV1 pad 2: Net-(R1-Pad1) -> Net-(D1-K)
- RV2 pad 2: Net-(R2-Pad1) -> Net-(D2-K)
Routing:
- net Net-(R1-Pad1): track 26.3 -> 0.00 mm
- net Net-(R2-Pad1): track 24.2 -> 0.00 mm
- net Net-(D1-K): track 20.5 -> 40.1 mm
- net Net-(D2-K): track 30.7 -> 50.2 mm
Other:
- board text added: "3V3"
- board text added: "5VIN"
- board text added: "ADC0+"
- board text added: "ADC0-"
- board text added: "ADC1+"
- board text added: "ADC1-"
- board text added: "COM+"
- board text added: "COM-"
- board text added: "GND"
- board text added: "IN0"
- board text added: "IN1"
- board text added: "IN2"
- board text added: "IN3"
- board text added: "IN4"
- board text added: "IN5"
- board text added: "OUT0"
- board text added: "OUT1"
- board text added: "OUT2"
- board text added: "OUT3"
- board text added: "OUT4"
- board text added: "OUT5"
- board text added: "PWM0"
- board text added: "PWM1"
